Commit message: arm cmake

File: arm/src/urdf/arm.plugins.xacro (robot description, xacro)
@@ -28,5 +28,5 @@
         <alwaysOn>true</alwaysOn>
         <updateRate>0.0</updateRate>
-        <cameraName>/arm_eden/camera</cameraName>
+        <cameraName>/arm/camera</cameraName>
         <imageTopicName>image_raw</imageTopicName>
         <cameraInfoTopicName>camera_info</cameraInfoTopicName>

File: arm/src/urdf/arm.xacro (robot description, xacro)
@@ -1,4 +1,4 @@
 <robot xmlns:xacro="http://www.ros.org/wiki/xacro" name="Eden">
-  <xacro:include filename="$(find arm_eden)/src/urdf/arm_eden.plugins.xacro" />
+  <xacro:include filename="$(find arm)/src/urdf/arm.plugins.xacro" />
   <xacro:property name="camera_size" value="0.02"/>
   <xacro:property name="camera_origin_x" value="0.065"/>
@@ -16,5 +16,5 @@
 <origin xyz="-0.06 4.48374e-18 0.06" rpy="-3.14159 1.5708 0" />
 <geometry>
-<mesh filename="package://arm_eden/src/meshes/skf_7208.stl"/>
+<mesh filename="package://arm/src/meshes/skf_7208.stl"/>
 </geometry>
 <material name="skf_7208_material">
@@ -25,5 +25,5 @@
 <origin xyz="-0.06 4.48374e-18 0.06" rpy="-3.14159 1.5708 0" />
 <geometry>
-<mesh filename="package://arm_eden/src/meshes/skf_7208.stl"/>
+<mesh filename="package://arm/src/meshes/skf_7208.stl"/>
 </geometry>
 <material name="skf_7208_material">
@@ -34,5 +34,5 @@
 <origin xyz="0.0025 1.00198e-14 0.052" rpy="-1.5708 -0 1.5708" />
 <geometry>
-<mesh filename="package://arm_eden/src/meshes/xl430.stl"/>
+<mesh filename="package://arm/src/meshes/xl430.stl"/>
 </geometry>
 <material name="xl430_material">
@@ -43,5 +43,5 @@
 <origin xyz="0.0025 1.00198e-14 0.052" rpy="-1.5708 -0 1.5708" />
 <geometry>
-<mesh filename="package://arm_eden/src/meshes/xl430.stl"/>
+<mesh filename="package://arm/src/meshes/xl430.stl"/>
 </geometry>
 <material name="xl430_material">
@@ -52,5 +52,5 @@
 <origin xyz="0.00249985 1.45751e-07 0.088" rpy="3.14159 -0 -1.5708" />
 <geometry>
-<mesh filename="package://arm_eden/src/meshes/small_gear_pilver.stl"/>
+<mesh filename="package://arm/src/meshes/small_gear_pilver.stl"/>
 </geometry>
 <material name="small_gear_pilver_material">
@@ -61,5 +61,5 @@
 <origin xyz="0.00249985 1.45751e-07 0.088" rpy="3.14159 -0 -1.5708" />
 <geometry>
-<mesh filename="package://arm_eden/src/meshes/small_gear_pilver.stl"/>
+<mesh filename="package://arm/src/meshes/small_gear_pilver.stl"/>
 </geometry>
 <material name="small_gear_pilver_material">
@@ -70,5 +70,5 @@
 <origin xyz="-0.06 4.48374e-18 0.026" rpy="-0 1.5708 0" />
 <geometry>
-<mesh filename="package://arm_eden/src/meshes/skf_7208.stl"/>
+<mesh filename="package://arm/src/meshes/skf_7208.stl"/>
 </geometry>
 <material name="skf_7208_material">
@@ -79,5 +79,5 @@
 <origin xyz="-0.06 4.48374e-18 0.026" rpy="-0 1.5708 0" />
 <geometry>
-<mesh filename="package://arm_eden/src/meshes/skf_7208.stl"/>
+<mesh filename="package://arm/src/meshes/skf_7208.stl"/>
 </geometry>
 <material name="skf_7208_material">
@@ -88,5 +88,5 @@
 <origin xyz="0.00249985 1.45751e-07 0.082" rpy="0 -0 -1.5708" />
 <geometry>
-<mesh filename="package://arm_eden/src/meshes/motor_link_xl.stl"/>
+<mesh filename="package://arm/src/meshes/motor_link_xl.stl"/>
 </geometry>
 <material name="motor_link_xl_material">
@@ -97,5 +97,5 @@
 <origin xyz="0.00249985 1.45751e-07 0.082" rpy="0 -0 -1.5708" />
 <geometry>
-<mesh filename="package://arm_eden/src/meshes/motor_link_xl.stl"/>
+<mesh filename="package://arm/src/meshes/motor_link_xl.stl"/>
 </geometry>
 <material name="motor_link_xl_material">
@@ -106,5 +106,5 @@
 <origin xyz="0 0 0" rpy="0 -0 0" />
 <geometry>
-<mesh filename="package://arm_eden/src/meshes/foundation.stl"/>
+<mesh filename="package://arm/src/meshes/foundation.stl"/>
 </geometry>
 <material name="foundation_material">
@@ -115,5 +115,5 @@
 <origin xyz="0 0 0" rpy="0 -0 0" />
 <geometry>
-<mesh filename="package://arm_eden/src/meshes/foundation.stl"/>
+<mesh filename="package://arm/src/meshes/foundation.stl"/>
 </geometry>
 <material name="foundation_material">
@@ -124,5 +124,5 @@
 <origin xyz="-6.93889e-18 0.115 0" rpy="0 -0 1.48691e-16" />
 <geometry>
-<mesh filename="package://arm_eden/src/meshes/wall_side.stl"/>
+<mesh filename="package://arm/src/meshes/wall_side.stl"/>
 </geometry>
 <material name="wall_side_material">
@@ -133,5 +133,5 @@
 <origin xyz="-6.93889e-18 0.115 0" rpy="0 -0 1.48691e-16" />
 <geometry>
-<mesh filename="package://arm_eden/src/meshes/wall_side.stl"/>
+<mesh filename="package://arm/src/meshes/wall_side.stl"/>
 </geometry>
 <material name="wall_side_material">
@@ -142,5 +142,5 @@
 <origin xyz="0 0 0" rpy="0 -0 0" />
 <geometry>
-<mesh filename="package://arm_eden/src/meshes/adapteur.stl"/>
+<mesh filename="package://arm/src/meshes/adapteur.stl"/>
 </geometry>
 <material name="adapteur_material">
@@ -151,5 +151,5 @@
 <origin xyz="0 0 0" rpy="0 -0 0" />
 <geometry>
-<mesh filename="package://arm_eden/src/meshes/adapteur.stl"/>
+<mesh filename="package://arm/src/meshes/adapteur.stl"/>
 </geometry>
 <material name="adapteur_material">
@@ -160,5 +160,5 @@
 <origin xyz="-6.93889e-18 6.93889e-18 0" rpy="0 -0 1.48691e-16" />
 <geometry>
-<mesh filename="package://arm_eden/src/meshes/wall_side.stl"/>
+<mesh filename="package://arm/src/meshes/wall_side.stl"/>
 </geometry>
 <material name="wall_side_material">
@@ -169,5 +169,5 @@
 <origin xyz="-6.93889e-18 6.93889e-18 0" rpy="0 -0 1.48691e-16" />
 <geometry>
-<mesh filename="package://arm_eden/src/meshes/wall_side.stl"/>
+<mesh filename="package://arm/src/meshes/wall_side.stl"/>
 </geometry>
 <material name="wall_side_material">
@@ -178,5 +178,5 @@
 <origin xyz="-2.77556e-17 -6.93889e-18 -8.67362e-19" rpy="0 -0 0" />
 <geometry>
-<mesh filename="package://arm_eden/src/meshes/wall_front.stl"/>
+<mesh filename="package://arm/src/meshes/wall_front.stl"/>
 </geometry>
 <material name="wall_front_material">
@@ -187,5 +187,5 @@
 <origin xyz="-2.77556e-17 -6.93889e-18 -8.67362e-19" rpy="0 -0 0" />
 <geometry>
-<mesh filename="package://arm_eden/src/meshes/wall_front.stl"/>
+<mesh filename="package://arm/src/meshes/wall_front.stl"/>
 </geometry>
 <material name="wall_front_material">
@@ -196,5 +196,5 @@
 <origin xyz="0 0 0" rpy="0 -0 0" />
 <geometry>
-<mesh filename="package://arm_eden/src/meshes/cover.stl"/>
+<mesh filename="package://arm/src/meshes/cover.stl"/>
 </geometry>
 <material name="cover_material">
@@ -205,5 +205,5 @@
 <origin xyz="0 0 0" rpy="0 -0 0" />
 <geometry>
-<mesh filename="package://arm_eden/src/meshes/cover.stl"/>
+<mesh filename="package://arm/src/meshes/cover.stl"/>
 </geometry>
 <material name="cover_material">
@@ -221,5 +221,5 @@
 <origin xyz="7.70372e-34 0 0.062" rpy="3.14159 -0 -3.14088e-49" />
 <geometry>
-<mesh filename="package://arm_eden/src/meshes/side_2.stl"/>
+<mesh filename="package://arm/src/meshes/side_2.stl"/>
 </geometry>
 <material name="side_2_material">
@@ -230,5 +230,5 @@
 <origin xyz="7.70372e-34 0 0.062" rpy="3.14159 -0 -3.14088e-49" />
 <geometry>
-<mesh filename="package://arm_eden/src/meshes/side_2.stl"/>
+<mesh filename="package://arm/src/meshes/side_2.stl"/>
 </geometry>
 <material name="side_2_material">
@@ -239,5 +239,5 @@
 <origin xyz="-0.0235 -1.01238e-14 -0.116" rpy="3.14159 -0 -3.14088e-49" />
 <geometry>
-<mesh filename="package://arm_eden/src/meshes/skf_7202.stl"/>
+<mesh filename="package://arm/src/meshes/skf_7202.stl"/>
 </geometry>
 <material name="skf_7202_material">
@@ -248,5 +248,5 @@
 <origin xyz="-0.0235 -1.01238e-14 -0.116" rpy="3.14159 -0 -3.14088e-49" />
 <geometry>
-<mesh filename="package://arm_eden/src/meshes/skf_7202.stl"/>
+<mesh filename="package://arm/src/meshes/skf_7202.stl"/>
 </geometry>
 <material name="skf_7202_material">
@@ -257,5 +257,5 @@
 <origin xyz="7.70372e-34 0 0.062" rpy="3.14159 -0 -3.14088e-49" />
 <geometry>
-<mesh filename="package://arm_eden/src/meshes/tree_base.stl"/>
+<mesh filename="package://arm/src/meshes/tree_base.stl"/>
 </geometry>
 <material name="tree_base_material">
@@ -266,5 +266,5 @@
 <origin xyz="7.70372e-34 0 0.062" rpy="3.14159 -0 -3.14088e-49" />
 <geometry>
-<mesh filename="package://arm_eden/src/meshes/tree_base.stl"/>
+<mesh filename="package://arm/src/meshes/tree_base.stl"/>
 </geometry>
 <material name="tree_base_material">
@@ -275,5 +275,5 @@
 <origin xyz="-0.109 -4.69555e-14 -0.013" rpy="3.14159 -0 -3.14088e-49" />
 <geometry>
-<mesh filename="package://arm_eden/src/meshes/big_gear_pilver.stl"/>
+<mesh filename="package://arm/src/meshes/big_gear_pilver.stl"/>
 </geometry>
 <material name="big_gear_pilver_material">
@@ -284,5 +284,5 @@
 <origin xyz="-0.109 -4.69555e-14 -0.013" rpy="3.14159 -0 -3.14088e-49" />
 <geometry>
-<mesh filename="package://arm_eden/src/meshes/big_gear_pilver.stl"/>
+<mesh filename="package://arm/src/meshes/big_gear_pilver.stl"/>
 </geometry>
 <material name="big_gear_pilver_material">
@@ -293,5 +293,5 @@
 <origin xyz="0.0235 1.02626e-14 -0.116" rpy="3.14159 -0 -3.14088e-49" />
 <geometry>
-<mesh filename="package://arm_eden/src/meshes/skf_7202.stl"/>
+<mesh filename="package://arm/src/meshes/skf_7202.stl"/>
 </geometry>
 <material name="skf_7202_material">
@@ -302,5 +302,5 @@
 <origin xyz="0.0235 1.02626e-14 -0.116" rpy="3.14159 -0 -3.14088e-49" />
 <geometry>
-<mesh filename="package://arm_eden/src/meshes/skf_7202.stl"/>
+<mesh filename="package://arm/src/meshes/skf_7202.stl"/>
 </geometry>
 <material name="skf_7202_material">
@@ -311,5 +311,5 @@
 <origin xyz="0.009 -0.06775 -0.12275" rpy="1.5708 1.5708 0" />
 <geometry>
-<mesh filename="package://arm_eden/src/meshes/xl430.stl"/>
+<mesh filename="package://arm/src/meshes/xl430.stl"/>
 </geometry>
 <material name="xl430_material">
@@ -320,5 +320,5 @@
 <origin xyz="0.009 -0.06775 -0.12275" rpy="1.5708 1.5708 0" />
 <geometry>
-<mesh filename="package://arm_eden/src/meshes/xl430.stl"/>
+<mesh filename="package://arm/src/meshes/xl430.stl"/>
 </geometry>
 <material name="xl430_material">
@@ -329,5 +329,5 @@
 <origin xyz="7.70372e-34 0 0.062" rpy="3.14159 -0 -3.14088e-49" />
 <geometry>
-<mesh filename="package://arm_eden/src/meshes/side.stl"/>
+<mesh filename="package://arm/src/meshes/side.stl"/>
 </geometry>
 <material name="side_material">
@@ -338,5 +338,5 @@
 <origin xyz="7.70372e-34 0 0.062" rpy="3.14159 -0 -3.14088e-49" />
 <geometry>
-<mesh filename="package://arm_eden/src/meshes/side.stl"/>
+<mesh filename="package://arm/src/meshes/side.stl"/>
 </geometry>
 <material name="side_material">
@@ -347,5 +347,5 @@
 <origin xyz="-0.016 -0.13525 -0.12275" rpy="1.5708 4.57546e-16 1.5708" />
 <geometry>
-<mesh filename="package://arm_eden/src/meshes/small_gear_shoulder.stl"/>
+<mesh filename="package://arm/src/meshes/small_gear_shoulder.stl"/>
 </geometry>
 <material name="small_gear_shoulder_material">
@@ -356,5 +356,5 @@
 <origin xyz="-0.016 -0.13525 -0.12275" rpy="1.5708 4.57546e-16 1.5708" />
 <geometry>
-<mesh filename="package://arm_eden/src/meshes/small_gear_shoulder.stl"/>
+<mesh filename="package://arm/src/meshes/small_gear_shoulder.stl"/>
 </geometry>
 <material name="small_gear_shoulder_material">
@@ -365,5 +365,5 @@
 <origin xyz="7.70372e-34 0 0.062" rpy="3.14159 -0 -3.14088e-49" />
 <geometry>
-<mesh filename="package://arm_eden/src/meshes/fixing_base_tree.stl"/>
+<mesh filename="package://arm/src/meshes/fixing_base_tree.stl"/>
 </geometry>
 <material name="fixing_base_tree_material">
@@ -374,5 +374,5 @@
 <origin xyz="7.70372e-34 0 0.062" rpy="3.14159 -0 -3.14088e-49" />
 <geometry>
-<mesh filename="package://arm_eden/src/meshes/fixing_base_tree.stl"/>
+<mesh filename="package://arm/src/meshes/fixing_base_tree.stl"/>
 </geometry>
 <material name="fixing_base_tree_material">
@@ -390,5 +390,5 @@
 <origin xyz="0 0 0.02" rpy="-1.5708 7.90622e-48 0" />
 <geometry>
-<mesh filename="package://arm_eden/src/meshes/arm_elbow.stl"/>
+<mesh filename="package://arm/src/meshes/arm_elbow.stl"/>
 </geometry>
 <material name="arm_elbow_material">
@@ -399,5 +399,5 @@
 <origin xyz="0 0 0.02" rpy="-1.5708 7.90622e-48 0" />
 <geometry>
-<mesh filename="package://arm_eden/src/meshes/arm_elbow.stl"/>
+<mesh filename="package://arm/src/meshes/arm_elbow.stl"/>
 </geometry>
 <material name="arm_elbow_material">
@@ -408,5 +408,5 @@
 <origin xyz="0 0 0.02" rpy="-1.5708 7.90622e-48 0" />
 <geometry>
-<mesh filename="package://arm_eden/src/meshes/tree_shoulder.stl"/>
+<mesh filename="package://arm/src/meshes/tree_shoulder.stl"/>
 </geometry>
 <material name="tree_shoulder_material">
@@ -417,5 +417,5 @@
 <origin xyz="0 0 0.02" rpy="-1.5708 7.90622e-48 0" />
 <geometry>
-<mesh filename="package://arm_eden/src/meshes/tree_shoulder.stl"/>
+<mesh filename="package://arm/src/meshes/tree_shoulder.stl"/>
 </geometry>
 <material name="tree_shoulder_material">
@@ -426,5 +426,5 @@
 <origin xyz="5.05151e-15 4.58366e-07 -0.008" rpy="-9.57715e-14 -2.09115e-13 -5.16254e-15" />
 <geometry>
-<mesh filename="package://arm_eden/src/meshes/big_gear_shoulder.stl"/>
+<mesh filename="package://arm/src/meshes/big_gear_shoulder.stl"/>
 </geometry>
 <material name="big_gear_shoulder_material">
@@ -435,5 +435,5 @@
 <origin xyz="5.05151e-15 4.58366e-07 -0.008" rpy="-9.57715e-14 -2.09115e-13 -5.16254e-15" />
 <geometry>
-<mesh filename="package://arm_eden/src/meshes/big_gear_shoulder.stl"/>
+<mesh filename="package://arm/src/meshes/big_gear_shoulder.stl"/>
 </geometry>
 <material name="big_gear_shoulder_material">
@@ -444,5 +444,5 @@
 <origin xyz="4.39926e-15 0.16 0.0115" rpy="-1.9984e-14 -1.5708 0" />
 <geometry>
-<mesh filename="package://arm_eden/src/meshes/skf_7202.stl"/>
+<mesh filename="package://arm/src/meshes/skf_7202.stl"/>
 </geometry>
 <material name="skf_7202_material">
@@ -453,5 +453,5 @@
 <origin xyz="4.39926e-15 0.16 0.0115" rpy="-1.9984e-14 -1.5708 0" />
 <geometry>
-<mesh filename="package://arm_eden/src/meshes/skf_7202.stl"/>
+<mesh filename="package://arm/src/meshes/skf_7202.stl"/>
 </geometry>
 <material name="skf_7202_material">
@@ -462,5 +462,5 @@
 <origin xyz="0 0 0.02" rpy="-1.5708 7.90622e-48 0" />
 <geometry>
-<mesh filename="package://arm_eden/src/meshes/fixing_shoulder_tree.stl"/>
+<mesh filename="package://arm/src/meshes/fixing_shoulder_tree.stl"/>
 </geometry>
 <material name="fixing_shoulder_tree_material">
@@ -471,5 +471,5 @@
 <origin xyz="0 0 0.02" rpy="-1.5708 7.90622e-48 0" />
 <geometry>
-<mesh filename="package://arm_eden/src/meshes/fixing_shoulder_tree.stl"/>
+<mesh filename="package://arm/src/meshes/fixing_shoulder_tree.stl"/>
 </geometry>
 <material name="fixing_shoulder_tree_material">
@@ -480,5 +480,5 @@
 <origin xyz="2.15453e-14 0.0969992 -0.033" rpy="1.5708 2.32728e-13 -3.14159" />
 <geometry>
-<mesh filename="package://arm_eden/src/meshes/xl430.stl"/>
+<mesh filename="package://arm/src/meshes/xl430.stl"/>
 </geometry>
 <material name="xl430_material">
@@ -489,5 +489,5 @@
 <origin xyz="2.15453e-14 0.0969992 -0.033" rpy="1.5708 2.32728e-13 -3.14159" />
 <geometry>
-<mesh filename="package://arm_eden/src/meshes/xl430.stl"/>
+<mesh filename="package://arm/src/meshes/xl430.stl"/>
 </geometry>
 <material name="xl430_material">
@@ -498,5 +498,5 @@
 <origin xyz="1.41831e-14 -3.60822e-16 -0.056" rpy="1.5708 2.32728e-13 -3.14159" />
 <geometry>
-<mesh filename="package://arm_eden/src/meshes/arm_elbow.stl"/>
+<mesh filename="package://arm/src/meshes/arm_elbow.stl"/>
 </geometry>
 <material name="arm_elbow_material">
@@ -507,5 +507,5 @@
 <origin xyz="1.41831e-14 -3.60822e-16 -0.056" rpy="1.5708 2.32728e-13 -3.14159" />
 <geometry>
-<mesh filename="package://arm_eden/src/meshes/arm_elbow.stl"/>
+<mesh filename="package://arm/src/meshes/arm_elbow.stl"/>
 </geometry>
 <material name="arm_elbow_material">
@@ -516,5 +516,5 @@
 <origin xyz="-1.4575e-07 0.156999 -0.063" rpy="3.14159 6.60176e-14 1.5708" />
 <geometry>
-<mesh filename="package://arm_eden/src/meshes/small_gear_elbow.stl"/>
+<mesh filename="package://arm/src/meshes/small_gear_elbow.stl"/>
 </geometry>
 <material name="small_gear_elbow_material">
@@ -525,5 +525,5 @@
 <origin xyz="-1.4575e-07 0.156999 -0.063" rpy="3.14159 6.60176e-14 1.5708" />
 <geometry>
-<mesh filename="package://arm_eden/src/meshes/small_gear_elbow.stl"/>
+<mesh filename="package://arm/src/meshes/small_gear_elbow.stl"/>
 </geometry>
 <material name="small_gear_elbow_material">
@@ -534,5 +534,5 @@
 <origin xyz="-1.4575e-07 0.0969993 -0.063" rpy="-3.14159 2.07477e-13 3.14159" />
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