Commit message: arm cmake

File: arm/src/urdf/robot.xacro (robot description, xacro)
@@ -1,4 +1,4 @@
 <robot xmlns:xacro="http://www.ros.org/wiki/xacro" name="Eden">
-  <xacro:include filename="$(find arm_eden)/src/urdf/materials.xacro" />
+  <xacro:include filename="$(find arm)/src/urdf/materials.xacro" />
 <link name="reference">
 <origin xyz="0 0 0" rpy="0 0 0" />
@@ -12,5 +12,5 @@
 <origin xyz="-0.06 4.48374e-18 0.06" rpy="-3.14159 1.5708 0" />
 <geometry>
-<mesh filename="package://arm_eden/src/meshes/skf_7208.stl"/>
+<mesh filename="package://arm/src/meshes/skf_7208.stl"/>
 </geometry>
 <material name="bearing_material" />
@@ -19,5 +19,5 @@
 <origin xyz="-0.06 4.48374e-18 0.06" rpy="-3.14159 1.5708 0" />
 <geometry>
-<mesh filename="package://arm_eden/src/meshes/skf_7208.stl"/>
+<mesh filename="package://arm/src/meshes/skf_7208.stl"/>
 </geometry>
 <material name="bearing_material" />
@@ -26,5 +26,5 @@
 <origin xyz="0.0025 1.00198e-14 0.052" rpy="-1.5708 -0 1.5708" />
 <geometry>
-<mesh filename="package://arm_eden/src/meshes/xl430.stl"/>
+<mesh filename="package://arm/src/meshes/xl430.stl"/>
 </geometry>
 <material name="xl430_material">
@@ -35,5 +35,5 @@
 <origin xyz="0.0025 1.00198e-14 0.052" rpy="-1.5708 -0 1.5708" />
 <geometry>
-<mesh filename="package://arm_eden/src/meshes/xl430.stl"/>
+<mesh filename="package://arm/src/meshes/xl430.stl"/>
 </geometry>
 <material name="xl430_material">
@@ -44,5 +44,5 @@
 <origin xyz="0.00249985 1.45751e-07 0.088" rpy="3.14159 -0 -1.5708" />
 <geometry>
-<mesh filename="package://arm_eden/src/meshes/small_gear_pilver.stl"/>
+<mesh filename="package://arm/src/meshes/small_gear_pilver.stl"/>
 </geometry>
 <material name="pvc" />
@@ -51,5 +51,5 @@
 <origin xyz="0.00249985 1.45751e-07 0.088" rpy="3.14159 -0 -1.5708" />
 <geometry>
-<mesh filename="package://arm_eden/src/meshes/small_gear_pilver.stl"/>
+<mesh filename="package://arm/src/meshes/small_gear_pilver.stl"/>
 </geometry>
 <material name="pvc" />
@@ -58,5 +58,5 @@
 <origin xyz="-0.06 4.48374e-18 0.026" rpy="-0 1.5708 0" />
 <geometry>
-<mesh filename="package://arm_eden/src/meshes/skf_7208.stl"/>
+<mesh filename="package://arm/src/meshes/skf_7208.stl"/>
 </geometry>
 <material name="bearing_material" />
@@ -65,5 +65,5 @@
 <origin xyz="-0.06 4.48374e-18 0.026" rpy="-0 1.5708 0" />
 <geometry>
-<mesh filename="package://arm_eden/src/meshes/skf_7208.stl"/>
+<mesh filename="package://arm/src/meshes/skf_7208.stl"/>
 </geometry>
 <material name="bearing_material" />
@@ -72,5 +72,5 @@
 <origin xyz="0.00249985 1.45751e-07 0.082" rpy="0 -0 -1.5708" />
 <geometry>
-<mesh filename="package://arm_eden/src/meshes/motor_link_xl.stl"/>
+<mesh filename="package://arm/src/meshes/motor_link_xl.stl"/>
 </geometry>
 <material name="pla" />
@@ -79,5 +79,5 @@
 <origin xyz="0.00249985 1.45751e-07 0.082" rpy="0 -0 -1.5708" />
 <geometry>
-<mesh filename="package://arm_eden/src/meshes/motor_link_xl.stl"/>
+<mesh filename="package://arm/src/meshes/motor_link_xl.stl"/>
 </geometry>
 <material name="pla" />
@@ -86,5 +86,5 @@
 <origin xyz="0 0 0" rpy="0 -0 0" />
 <geometry>
-<mesh filename="package://arm_eden/src/meshes/foundation.stl"/>
+<mesh filename="package://arm/src/meshes/foundation.stl"/>
 </geometry>
 <material name="wood" />
@@ -93,5 +93,5 @@
 <origin xyz="0 0 0" rpy="0 -0 0" />
 <geometry>
-<mesh filename="package://arm_eden/src/meshes/foundation.stl"/>
+<mesh filename="package://arm/src/meshes/foundation.stl"/>
 </geometry>
 <material name="wood" />
@@ -100,5 +100,5 @@
 <origin xyz="-6.93889e-18 0.115 0" rpy="0 -0 1.48691e-16" />
 <geometry>
-<mesh filename="package://arm_eden/src/meshes/wall_side.stl"/>
+<mesh filename="package://arm/src/meshes/wall_side.stl"/>
 </geometry>
 <material name="wood" />
@@ -107,5 +107,5 @@
 <origin xyz="-6.93889e-18 0.115 0" rpy="0 -0 1.48691e-16" />
 <geometry>
-<mesh filename="package://arm_eden/src/meshes/wall_side.stl"/>
+<mesh filename="package://arm/src/meshes/wall_side.stl"/>
 </geometry>
 <material name="wood" />
@@ -114,5 +114,5 @@
 <origin xyz="0 0 0" rpy="0 -0 0" />
 <geometry>
-<mesh filename="package://arm_eden/src/meshes/adapteur.stl"/>
+<mesh filename="package://arm/src/meshes/adapteur.stl"/>
 </geometry>
 <material name="pla" />
@@ -121,5 +121,5 @@
 <origin xyz="0 0 0" rpy="0 -0 0" />
 <geometry>
-<mesh filename="package://arm_eden/src/meshes/adapteur.stl"/>
+<mesh filename="package://arm/src/meshes/adapteur.stl"/>
 </geometry>
 <material name="pla" />
@@ -128,5 +128,5 @@
 <origin xyz="-6.93889e-18 6.93889e-18 0" rpy="0 -0 1.48691e-16" />
 <geometry>
-<mesh filename="package://arm_eden/src/meshes/wall_side.stl"/>
+<mesh filename="package://arm/src/meshes/wall_side.stl"/>
 </geometry>
 <material name="wood" />
@@ -135,5 +135,5 @@
 <origin xyz="-6.93889e-18 6.93889e-18 0" rpy="0 -0 1.48691e-16" />
 <geometry>
-<mesh filename="package://arm_eden/src/meshes/wall_side.stl"/>
+<mesh filename="package://arm/src/meshes/wall_side.stl"/>
 </geometry>
 <material name="wood" />
@@ -142,5 +142,5 @@
 <origin xyz="-2.77556e-17 -6.93889e-18 -8.67362e-19" rpy="0 -0 0" />
 <geometry>
-<mesh filename="package://arm_eden/src/meshes/wall_front.stl"/>
+<mesh filename="package://arm/src/meshes/wall_front.stl"/>
 </geometry>
 <material name="wood" />
@@ -149,5 +149,5 @@
 <origin xyz="-2.77556e-17 -6.93889e-18 -8.67362e-19" rpy="0 -0 0" />
 <geometry>
-<mesh filename="package://arm_eden/src/meshes/wall_front.stl"/>
+<mesh filename="package://arm/src/meshes/wall_front.stl"/>
 </geometry>
 <material name="wood" />
@@ -156,5 +156,5 @@
 <origin xyz="0 0 0" rpy="0 -0 0" />
 <geometry>
-<mesh filename="package://arm_eden/src/meshes/cover.stl"/>
+<mesh filename="package://arm/src/meshes/cover.stl"/>
 </geometry>
 <material name="wood" />
@@ -163,5 +163,5 @@
 <origin xyz="0 0 0" rpy="0 -0 0" />
 <geometry>
-<mesh filename="package://arm_eden/src/meshes/cover.stl"/>
+<mesh filename="package://arm/src/meshes/cover.stl"/>
 </geometry>
 <material name="wood" />
@@ -177,5 +177,5 @@
 <origin xyz="7.70372e-34 0 0.062" rpy="3.14159 -0 -3.14088e-49" />
 <geometry>
-<mesh filename="package://arm_eden/src/meshes/side_2.stl"/>
+<mesh filename="package://arm/src/meshes/side_2.stl"/>
 </geometry>
 <material name="pvc" />
@@ -184,5 +184,5 @@
 <origin xyz="7.70372e-34 0 0.062" rpy="3.14159 -0 -3.14088e-49" />
 <geometry>
-<mesh filename="package://arm_eden/src/meshes/side_2.stl"/>
+<mesh filename="package://arm/src/meshes/side_2.stl"/>
 </geometry>
 <material name="pvc" />
@@ -191,5 +191,5 @@
 <origin xyz="-0.0235 -1.01238e-14 -0.116" rpy="3.14159 -0 -3.14088e-49" />
 <geometry>
-<mesh filename="package://arm_eden/src/meshes/skf_7202.stl"/>
+<mesh filename="package://arm/src/meshes/skf_7202.stl"/>
 </geometry>
 <material name="bearing_material" />
@@ -198,5 +198,5 @@
 <origin xyz="-0.0235 -1.01238e-14 -0.116" rpy="3.14159 -0 -3.14088e-49" />
 <geometry>
-<mesh filename="package://arm_eden/src/meshes/skf_7202.stl"/>
+<mesh filename="package://arm/src/meshes/skf_7202.stl"/>
 </geometry>
 <material name="bearing_material" />
@@ -205,5 +205,5 @@
 <origin xyz="7.70372e-34 0 0.062" rpy="3.14159 -0 -3.14088e-49" />
 <geometry>
-<mesh filename="package://arm_eden/src/meshes/tree_base.stl"/>
+<mesh filename="package://arm/src/meshes/tree_base.stl"/>
 </geometry>
 <material name="pla" />
@@ -212,5 +212,5 @@
 <origin xyz="7.70372e-34 0 0.062" rpy="3.14159 -0 -3.14088e-49" />
 <geometry>
-<mesh filename="package://arm_eden/src/meshes/tree_base.stl"/>
+<mesh filename="package://arm/src/meshes/tree_base.stl"/>
 </geometry>
 <material name="pla" />
@@ -219,5 +219,5 @@
 <origin xyz="-0.109 -4.69555e-14 -0.013" rpy="3.14159 -0 -3.14088e-49" />
 <geometry>
-<mesh filename="package://arm_eden/src/meshes/big_gear_pilver.stl"/>
+<mesh filename="package://arm/src/meshes/big_gear_pilver.stl"/>
 </geometry>
 <material name="pvc" />
@@ -226,5 +226,5 @@
 <origin xyz="-0.109 -4.69555e-14 -0.013" rpy="3.14159 -0 -3.14088e-49" />
 <geometry>
-<mesh filename="package://arm_eden/src/meshes/big_gear_pilver.stl"/>
+<mesh filename="package://arm/src/meshes/big_gear_pilver.stl"/>
 </geometry>
 <material name="pvc" />
@@ -233,5 +233,5 @@
 <origin xyz="0.0235 1.02626e-14 -0.116" rpy="3.14159 -0 -3.14088e-49" />
 <geometry>
-<mesh filename="package://arm_eden/src/meshes/skf_7202.stl"/>
+<mesh filename="package://arm/src/meshes/skf_7202.stl"/>
 </geometry>
 <material name="bearing_material" />
@@ -240,5 +240,5 @@
 <origin xyz="0.0235 1.02626e-14 -0.116" rpy="3.14159 -0 -3.14088e-49" />
 <geometry>
-<mesh filename="package://arm_eden/src/meshes/skf_7202.stl"/>
+<mesh filename="package://arm/src/meshes/skf_7202.stl"/>
 </geometry>
 <material name="bearing_material" />
@@ -247,5 +247,5 @@
 <origin xyz="0.009 -0.06775 -0.12275" rpy="1.5708 1.5708 0" />
 <geometry>
-<mesh filename="package://arm_eden/src/meshes/xl430.stl"/>
+<mesh filename="package://arm/src/meshes/xl430.stl"/>
 </geometry>
 <material name="xl430_material">
@@ -256,5 +256,5 @@
 <origin xyz="0.009 -0.06775 -0.12275" rpy="1.5708 1.5708 0" />
 <geometry>
-<mesh filename="package://arm_eden/src/meshes/xl430.stl"/>
+<mesh filename="package://arm/src/meshes/xl430.stl"/>
 </geometry>
 <material name="xl430_material">
@@ -265,5 +265,5 @@
 <origin xyz="7.70372e-34 0 0.062" rpy="3.14159 -0 -3.14088e-49" />
 <geometry>
-<mesh filename="package://arm_eden/src/meshes/side.stl"/>
+<mesh filename="package://arm/src/meshes/side.stl"/>
 </geometry>
 <material name="pvc" />
@@ -272,5 +272,5 @@
 <origin xyz="7.70372e-34 0 0.062" rpy="3.14159 -0 -3.14088e-49" />
 <geometry>
-<mesh filename="package://arm_eden/src/meshes/side.stl"/>
+<mesh filename="package://arm/src/meshes/side.stl"/>
 </geometry>
 <material name="pvc" />
@@ -279,5 +279,5 @@
 <origin xyz="-0.016 -0.13525 -0.12275" rpy="1.5708 4.57546e-16 1.5708" />
 <geometry>
-<mesh filename="package://arm_eden/src/meshes/small_gear_shoulder.stl"/>
+<mesh filename="package://arm/src/meshes/small_gear_shoulder.stl"/>
 </geometry>
 <material name="pvc" />
@@ -286,5 +286,5 @@
 <origin xyz="-0.016 -0.13525 -0.12275" rpy="1.5708 4.57546e-16 1.5708" />
 <geometry>
-<mesh filename="package://arm_eden/src/meshes/small_gear_shoulder.stl"/>
+<mesh filename="package://arm/src/meshes/small_gear_shoulder.stl"/>
 </geometry>
 <material name="pvc" />
@@ -293,5 +293,5 @@
 <origin xyz="7.70372e-34 0 0.062" rpy="3.14159 -0 -3.14088e-49" />
 <geometry>
-<mesh filename="package://arm_eden/src/meshes/fixing_base_tree.stl"/>
+<mesh filename="package://arm/src/meshes/fixing_base_tree.stl"/>
 </geometry>
 <material name="pla" />
@@ -300,5 +300,5 @@
 <origin xyz="7.70372e-34 0 0.062" rpy="3.14159 -0 -3.14088e-49" />
 <geometry>
-<mesh filename="package://arm_eden/src/meshes/fixing_base_tree.stl"/>
+<mesh filename="package://arm/src/meshes/fixing_base_tree.stl"/>
 </geometry>
 <material name="pla" />
@@ -314,5 +314,5 @@
 <origin xyz="0 0 0.02" rpy="-1.5708 7.90622e-48 0" />
 <geometry>
-<mesh filename="package://arm_eden/src/meshes/arm_elbow.stl"/>
+<mesh filename="package://arm/src/meshes/arm_elbow.stl"/>
 </geometry>
 <material name="pvc" />
@@ -321,5 +321,5 @@
 <origin xyz="0 0 0.02" rpy="-1.5708 7.90622e-48 0" />
 <geometry>
-<mesh filename="package://arm_eden/src/meshes/arm_elbow.stl"/>
+<mesh filename="package://arm/src/meshes/arm_elbow.stl"/>
 </geometry>
 <material name="pvc" />
@@ -328,5 +328,5 @@
 <origin xyz="0 0 0.02" rpy="-1.5708 7.90622e-48 0" />
 <geometry>
-<mesh filename="package://arm_eden/src/meshes/tree_shoulder.stl"/>
+<mesh filename="package://arm/src/meshes/tree_shoulder.stl"/>
 </geometry>
 <material name="pla" />
@@ -335,5 +335,5 @@
 <origin xyz="0 0 0.02" rpy="-1.5708 7.90622e-48 0" />
 <geometry>
-<mesh filename="package://arm_eden/src/meshes/tree_shoulder.stl"/>
+<mesh filename="package://arm/src/meshes/tree_shoulder.stl"/>
 </geometry>
 <material name="pla" />
@@ -342,5 +342,5 @@
 <origin xyz="5.05151e-15 4.58366e-07 -0.008" rpy="-9.57715e-14 -2.09115e-13 -5.16254e-15" />
 <geometry>
-<mesh filename="package://arm_eden/src/meshes/big_gear_shoulder.stl"/>
+<mesh filename="package://arm/src/meshes/big_gear_shoulder.stl"/>
 </geometry>
 <material name="pvc" />
@@ -349,5 +349,5 @@
 <origin xyz="5.05151e-15 4.58366e-07 -0.008" rpy="-9.57715e-14 -2.09115e-13 -5.16254e-15" />
 <geometry>
-<mesh filename="package://arm_eden/src/meshes/big_gear_shoulder.stl"/>
+<mesh filename="package://arm/src/meshes/big_gear_shoulder.stl"/>
 </geometry>
 <material name="pvc" />
@@ -356,5 +356,5 @@
 <origin xyz="4.39926e-15 0.16 0.0115" rpy="-1.9984e-14 -1.5708 0" />
 <geometry>
-<mesh filename="package://arm_eden/src/meshes/skf_7202.stl"/>
+<mesh filename="package://arm/src/meshes/skf_7202.stl"/>
 </geometry>
 <material name="bearing_material" />
@@ -363,5 +363,5 @@
 <origin xyz="4.39926e-15 0.16 0.0115" rpy="-1.9984e-14 -1.5708 0" />
 <geometry>
-<mesh filename="package://arm_eden/src/meshes/skf_7202.stl"/>
+<mesh filename="package://arm/src/meshes/skf_7202.stl"/>
 </geometry>
 <material name="bearing_material" />
@@ -370,5 +370,5 @@
 <origin xyz="0 0 0.02" rpy="-1.5708 7.90622e-48 0" />
 <geometry>
-<mesh filename="package://arm_eden/src/meshes/fixing_shoulder_tree.stl"/>
+<mesh filename="package://arm/src/meshes/fixing_shoulder_tree.stl"/>
 </geometry>
 <material name="pla" />
@@ -377,5 +377,5 @@
 <origin xyz="0 0 0.02" rpy="-1.5708 7.90622e-48 0" />
 <geometry>
-<mesh filename="package://arm_eden/src/meshes/fixing_shoulder_tree.stl"/>
+<mesh filename="package://arm/src/meshes/fixing_shoulder_tree.stl"/>
 </geometry>
 <material name="pla" />
@@ -384,5 +384,5 @@
 <origin xyz="2.15453e-14 0.0969992 -0.033" rpy="1.5708 2.32728e-13 -3.14159" />
 <geometry>
-<mesh filename="package://arm_eden/src/meshes/xl430.stl"/>
+<mesh filename="package://arm/src/meshes/xl430.stl"/>
 </geometry>
 <material name="xl430_material">
@@ -393,5 +393,5 @@
 <origin xyz="2.15453e-14 0.0969992 -0.033" rpy="1.5708 2.32728e-13 -3.14159" />
 <geometry>
-<mesh filename="package://arm_eden/src/meshes/xl430.stl"/>
+<mesh filename="package://arm/src/meshes/xl430.stl"/>
 </geometry>
 <material name="xl430_material">
@@ -402,5 +402,5 @@
 <origin xyz="1.41831e-14 -3.60822e-16 -0.056" rpy="1.5708 2.32728e-13 -3.14159" />
 <geometry>
-<mesh filename="package://arm_eden/src/meshes/arm_elbow.stl"/>
+<mesh filename="package://arm/src/meshes/arm_elbow.stl"/>
 </geometry>
 <material name="pvc" />
@@ -409,5 +409,5 @@
 <origin xyz="1.41831e-14 -3.60822e-16 -0.056" rpy="1.5708 2.32728e-13 -3.14159" />
 <geometry>
-<mesh filename="package://arm_eden/src/meshes/arm_elbow.stl"/>
+<mesh filename="package://arm/src/meshes/arm_elbow.stl"/>
 </geometry>
 <material name="pvc" />
@@ -416,5 +416,5 @@
 <origin xyz="-1.4575e-07 0.156999 -0.063" rpy="3.14159 6.60176e-14 1.5708" />
 <geometry>
-<mesh filename="package://arm_eden/src/meshes/small_gear_elbow.stl"/>
+<mesh filename="package://arm/src/meshes/small_gear_elbow.stl"/>
 </geometry>
 <material name="pvc" />
@@ -423,5 +423,5 @@
 <origin xyz="-1.4575e-07 0.156999 -0.063" rpy="3.14159 6.60176e-14 1.5708" />
 <geometry>
-<mesh filename="package://arm_eden/src/meshes/small_gear_elbow.stl"/>
+<mesh filename="package://arm/src/meshes/small_gear_elbow.stl"/>
 </geometry>
 <material name="pvc" />
@@ -430,5 +430,5 @@
 <origin xyz="-1.4575e-07 0.0969993 -0.063" rpy="-3.14159 2.07477e-13 3.14159" />
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