Commit message: urdf correction

File: arm/src/urdf/materials.xacro (robot description, xacro)
@@ -1,15 +1,21 @@
 <?xml version="1.0"?>
 <robot>
-<material name="bearing_material">
-<color rgba="0.647059 0.647059 0.647059 1.0"/>
-</material>
-<material name="pvc">
-<color rgba="0.917647 0.917647 0.917647 1.0"/>
-</material>
-<material name="wood">
-<color rgba="0.917647 0.72549 0.490196 1.0"/>
-</material>
-<material name="pla">
-<color rgba="0.87451 0.447059 0.317647 1.0"/>
-</material>
+    <material name="bearing_material">
+        <color rgba="0.647059 0.647059 0.647059 1.0"/>
+    </material>
+    <material name="xl430_material">
+        <color rgba="0.501961 0.501961 0.501961 1.0"/>
+    </material>
+    <material name="pvc">
+        <color rgba="0.917647 0.917647 0.917647 1.0"/>
+    </material>
+    <material name="plywood">
+        <color rgba="0.917647 0.72549 0.490196 1.0"/>
+    </material>
+    <material name="pla">
+        <color rgba="0.87451 0.447059 0.317647 1.0"/>
+    </material>
+    <material name="steel">
+        <color rgba="0.615686 0.811765 0.929412 1.0"/>
+    </material>
 </robot>

File: arm/src/urdf/robot.xacro (robot description, xacro)
@@ -1,2 +1,8 @@
+<!--
+unit :
+    - distance : m
+    - mass : kg
+    - time : s
+ -->
 <robot xmlns:xacro="http://www.ros.org/wiki/xacro" name="Eden">
   <xacro:include filename="$(find arm)/src/urdf/materials.xacro" />
@@ -24,7 +30,5 @@
                 <mesh filename="package://arm/src/meshes/xl430.stl"/>
             </geometry>
-            <material name="xl430_material">
-                <color rgba="0.501961 0.501961 0.501961 1.0"/>
-            </material>
+            <material name="xl430_material"/>
         </visual>
         <collision>
@@ -33,7 +37,5 @@
                 <mesh filename="package://arm/src/meshes/xl430.stl"/>
             </geometry>
-            <material name="xl430_material">
-                <color rgba="0.501961 0.501961 0.501961 1.0"/>
-            </material>
+            <material name="xl430_material"/>
         </collision>
         <visual>
@@ -43,5 +45,5 @@
             </geometry>
             <material name="pvc"/>
-            </visual>
+        </visual>
         <collision>
             <origin xyz="0.00249985 1.45751e-07 0.088" rpy="3.14159 -0 -1.5708" />
@@ -82,14 +84,14 @@
             <origin xyz="0 0 0" rpy="0 -0 0" />
             <geometry>
-                <mesh filename="package://arm/src/meshes/foundation.stl"/>
-            </geometry>
-            <material name="wood"/>
+                <mesh filename="package://arm/src/meshes/bottom.stl"/>
+            </geometry>
+            <material name="plywood"/>
         </visual>
         <collision>
             <origin xyz="0 0 0" rpy="0 -0 0" />
             <geometry>
-                <mesh filename="package://arm/src/meshes/foundation.stl"/>
-            </geometry>
-            <material name="wood"/>
+                <mesh filename="package://arm/src/meshes/bottom.stl"/>
+            </geometry>
+            <material name="plywood"/>
         </collision>
         <visual>
@@ -98,5 +100,5 @@
                 <mesh filename="package://arm/src/meshes/wall_side.stl"/>
             </geometry>
-            <material name="wood"/>
+            <material name="plywood"/>
         </visual>
         <collision>
@@ -105,5 +107,5 @@
                 <mesh filename="package://arm/src/meshes/wall_side.stl"/>
             </geometry>
-            <material name="wood"/>
+            <material name="plywood"/>
         </collision>
         <visual>
@@ -126,5 +128,5 @@
                 <mesh filename="package://arm/src/meshes/wall_side.stl"/>
             </geometry>
-            <material name="wood"/>
+            <material name="plywood"/>
         </visual>
         <collision>
@@ -133,5 +135,5 @@
                 <mesh filename="package://arm/src/meshes/wall_side.stl"/>
             </geometry>
-            <material name="wood"/>
+            <material name="plywood"/>
         </collision>
         <visual>
@@ -140,5 +142,5 @@
                 <mesh filename="package://arm/src/meshes/wall_front.stl"/>
             </geometry>
-            <material name="wood"/>
+            <material name="plywood"/>
         </visual>
         <collision>
@@ -147,19 +149,19 @@
                 <mesh filename="package://arm/src/meshes/wall_front.stl"/>
             </geometry>
-            <material name="wood"/>
-        </collision>
-            <visual>
+            <material name="plywood"/>
+        </collision>
+        <visual>
             <origin xyz="0 0 0" rpy="0 -0 0" />
             <geometry>
-                <mesh filename="package://arm/src/meshes/cover.stl"/>
-            </geometry>
-            <material name="wood"/>
+                <mesh filename="package://arm/src/meshes/top.stl"/>
+            </geometry>
+            <material name="plywood"/>
         </visual>
         <collision>
             <origin xyz="0 0 0" rpy="0 -0 0" />
             <geometry>
-                <mesh filename="package://arm/src/meshes/cover.stl"/>
-            </geometry>
-            <material name="wood"/>
+                <mesh filename="package://arm/src/meshes/top.stl"/>
+            </geometry>
+            <material name="plywood"/>
         </collision>
         <inertial>
@@ -171,5 +173,5 @@
     <link name="hip">
         <visual>
-            <origin xyz="7.70372e-34 0 0.062" rpy="3.14159 -0 -3.14088e-49" />
+            <origin xyz="-6.93889e-18 0 0.062" rpy="-3.14159 -0 4.01069e-70" />
             <geometry>
                 <mesh filename="package://arm/src/meshes/side_2.stl"/>
@@ -178,5 +180,5 @@
         </visual>
         <collision>
-            <origin xyz="7.70372e-34 0 0.062" rpy="3.14159 -0 -3.14088e-49" />
+            <origin xyz="-6.93889e-18 0 0.062" rpy="-3.14159 -0 4.01069e-70" />
             <geometry>
                 <mesh filename="package://arm/src/meshes/side_2.stl"/>
@@ -185,19 +187,19 @@
         </collision>
         <visual>
-            <origin xyz="-0.0235 -1.01238e-14 -0.116" rpy="3.14159 -0 -3.14088e-49" />
-            <geometry>
-                <mesh filename="package://arm/src/meshes/skf_7202.stl"/>
-            </geometry>
-            <material name="bearing_material"/>
-        </visual>
-        <collision>
-            <origin xyz="-0.0235 -1.01238e-14 -0.116" rpy="3.14159 -0 -3.14088e-49" />
-            <geometry>
-                <mesh filename="package://arm/src/meshes/skf_7202.stl"/>
-            </geometry>
-            <material name="bearing_material"/>
-        </collision>
-        <visual>
-            <origin xyz="7.70372e-34 0 0.062" rpy="3.14159 -0 -3.14088e-49" />
+            <origin xyz="-0.0235 2.08167e-17 -0.116" rpy="-3.14159 -0 4.01069e-70" />
+            <geometry>
+                <mesh filename="package://arm/src/meshes/skf_7202.stl"/>
+            </geometry>
+            <material name="bearing_material"/>
+        </visual>
+        <collision>
+            <origin xyz="-0.0235 2.08167e-17 -0.116" rpy="-3.14159 -0 4.01069e-70" />
+            <geometry>
+                <mesh filename="package://arm/src/meshes/skf_7202.stl"/>
+            </geometry>
+            <material name="bearing_material"/>
+        </collision>
+        <visual>
+            <origin xyz="0 0 0.062" rpy="-3.14159 -0 4.01069e-70" />
             <geometry>
                 <mesh filename="package://arm/src/meshes/tree_base.stl"/>
@@ -206,5 +208,5 @@
         </visual>
         <collision>
-            <origin xyz="7.70372e-34 0 0.062" rpy="3.14159 -0 -3.14088e-49" />
+            <origin xyz="0 0 0.062" rpy="-3.14159 -0 4.01069e-70" />
             <geometry>
                 <mesh filename="package://arm/src/meshes/tree_base.stl"/>
@@ -213,5 +215,5 @@
         </collision>
         <visual>
-            <origin xyz="-0.109 -4.69555e-14 -0.013" rpy="3.14159 -0 -3.14088e-49" />
+            <origin xyz="-0.109 -1.38778e-17 -0.013" rpy="-3.14159 -0 4.01069e-70" />
             <geometry>
                 <mesh filename="package://arm/src/meshes/big_gear_pelvis.stl"/>
@@ -220,5 +222,5 @@
         </visual>
         <collision>
-            <origin xyz="-0.109 -4.69555e-14 -0.013" rpy="3.14159 -0 -3.14088e-49" />
+            <origin xyz="-0.109 -1.38778e-17 -0.013" rpy="-3.14159 -0 4.01069e-70" />
             <geometry>
                 <mesh filename="package://arm/src/meshes/big_gear_pelvis.stl"/>
@@ -227,12 +229,12 @@
         </collision>
         <visual>
-            <origin xyz="0.0235 1.02626e-14 -0.116" rpy="3.14159 -0 -3.14088e-49" />
-            <geometry>
-                <mesh filename="package://arm/src/meshes/skf_7202.stl"/>
-            </geometry>
-            <material name="bearing_material"/>
-        </visual>
-        <collision>
-            <origin xyz="0.0235 1.02626e-14 -0.116" rpy="3.14159 -0 -3.14088e-49" />
+            <origin xyz="0.0235 2.08167e-17 -0.116" rpy="-3.14159 -0 4.01069e-70" />
+            <geometry>
+                <mesh filename="package://arm/src/meshes/skf_7202.stl"/>
+            </geometry>
+            <material name="bearing_material"/>
+        </visual>
+        <collision>
+            <origin xyz="0.0235 2.08167e-17 -0.116" rpy="-3.14159 -0 4.01069e-70" />
             <geometry>
                 <mesh filename="package://arm/src/meshes/skf_7202.stl"/>
@@ -245,7 +247,5 @@
                 <mesh filename="package://arm/src/meshes/xl430.stl"/>
             </geometry>
-            <material name="xl430_material">
-                <color rgba="0.501961 0.501961 0.501961 1.0"/>
-            </material>
+            <material name="xl430_material"/>
         </visual>
         <collision>
@@ -254,10 +254,8 @@
                 <mesh filename="package://arm/src/meshes/xl430.stl"/>
             </geometry>
-            <material name="xl430_material">
-                <color rgba="0.501961 0.501961 0.501961 1.0"/>
-            </material>
-        </collision>
-        <visual>
-            <origin xyz="7.70372e-34 0 0.062" rpy="3.14159 -0 -3.14088e-49" />
+            <material name="xl430_material"/>
+        </collision>
+        <visual>
+            <origin xyz="0 0 0.062" rpy="-3.14159 -0 4.01069e-70" />
             <geometry>
                 <mesh filename="package://arm/src/meshes/side.stl"/>
@@ -266,5 +264,5 @@
         </visual>
         <collision>
-            <origin xyz="7.70372e-34 0 0.062" rpy="3.14159 -0 -3.14088e-49" />
+            <origin xyz="0 0 0.062" rpy="-3.14159 -0 4.01069e-70" />
             <geometry>
                 <mesh filename="package://arm/src/meshes/side.stl"/>
@@ -273,5 +271,5 @@
         </collision>
         <visual>
-            <origin xyz="-0.016 -0.13525 -0.12275" rpy="1.5708 4.57546e-16 1.5708" />
+            <origin xyz="-0.016 -0.13525 -0.12275" rpy="1.5708 -6.37237e-58 1.5708" />
             <geometry>
                 <mesh filename="package://arm/src/meshes/small_gear_shoulder.stl"/>
@@ -280,5 +278,5 @@
         </visual>
         <collision>
-            <origin xyz="-0.016 -0.13525 -0.12275" rpy="1.5708 4.57546e-16 1.5708" />
+            <origin xyz="-0.016 -0.13525 -0.12275" rpy="1.5708 -6.37237e-58 1.5708" />
             <geometry>
                 <mesh filename="package://arm/src/meshes/small_gear_shoulder.stl"/>
@@ -287,5 +285,5 @@
         </collision>
         <visual>
-            <origin xyz="7.70372e-34 0 0.062" rpy="3.14159 -0 -3.14088e-49" />
+            <origin xyz="0 0 0.062" rpy="-3.14159 -0 4.01069e-70" />
             <geometry>
                 <mesh filename="package://arm/src/meshes/fixing_base_tree.stl"/>
@@ -294,5 +292,5 @@
         </visual>
         <collision>
-            <origin xyz="7.70372e-34 0 0.062" rpy="3.14159 -0 -3.14088e-49" />
+            <origin xyz="0 0 0.062" rpy="-3.14159 -0 4.01069e-70" />
             <geometry>
                 <mesh filename="package://arm/src/meshes/fixing_base_tree.stl"/>
@@ -308,19 +306,19 @@
     <link name="humerus">
         <visual>
-            <origin xyz="0 0 0.04" rpy="-1.5708 7.90622e-48 0" />
-            <geometry>
-                <mesh filename="package://arm/src/meshes/arm_elbow.stl"/>
-            </geometry>
-            <material name="pvc"/>
-        </visual>
-        <collision>
-            <origin xyz="0 0 0.04" rpy="-1.5708 7.90622e-48 0" />
-            <geometry>
-                <mesh filename="package://arm/src/meshes/arm_elbow.stl"/>
-            </geometry>
-            <material name="pvc"/>
-        </collision>
-        <visual>
-            <origin xyz="0 0 0.02" rpy="-1.5708 7.90622e-48 0" />
+            <origin xyz="6.93889e-18 0 0.02" rpy="-1.5708 -9.99986e-31 0" />
+            <geometry>
+                <mesh filename="package://arm/src/meshes/humerus.stl"/>
+            </geometry>
+            <material name="pvc"/>
+        </visual>
+        <collision>
+            <origin xyz="6.93889e-18 0 0.02" rpy="-1.5708 -9.99986e-31 0" />
+            <geometry>
+                <mesh filename="package://arm/src/meshes/humerus.stl"/>
+            </geometry>
+            <material name="pvc"/>
+        </collision>
+        <visual>
+            <origin xyz="6.93889e-18 0 0.02" rpy="-1.5708 -9.99986e-31 0" />
             <geometry>
                 <mesh filename="package://arm/src/meshes/tree_shoulder.stl"/>
@@ -329,5 +327,5 @@
         </visual>
         <collision>
-            <origin xyz="0 0 0.02" rpy="-1.5708 7.90622e-48 0" />
+            <origin xyz="6.93889e-18 0 0.02" rpy="-1.5708 -9.99986e-31 0" />
             <geometry>
                 <mesh filename="package://arm/src/meshes/tree_shoulder.stl"/>
@@ -336,5 +334,5 @@
         </collision>
         <visual>
-            <origin xyz="5.05151e-15 4.58366e-07 -0.008" rpy="-9.57715e-14 -2.09115e-13 -5.16254e-15" />
+            <origin xyz="0 4.58366e-07 -0.008" rpy="0 -9.99986e-31 0" />
             <geometry>
                 <mesh filename="package://arm/src/meshes/big_gear_shoulder.stl"/>
@@ -343,5 +341,5 @@
         </visual>
         <collision>
-            <origin xyz="5.05151e-15 4.58366e-07 -0.008" rpy="-9.57715e-14 -2.09115e-13 -5.16254e-15" />
+            <origin xyz="0 4.58366e-07 -0.008" rpy="0 -9.99986e-31 0" />
             <geometry>
                 <mesh filename="package://arm/src/meshes/big_gear_shoulder.stl"/>
@@ -350,19 +348,19 @@
         </collision>
         <visual>
-            <origin xyz="4.39926e-15 0.16 0.0115" rpy="-1.9984e-14 -1.5708 0" />
-            <geometry>
-                <mesh filename="package://arm/src/meshes/skf_7202.stl"/>
-            </geometry>
-            <material name="bearing_material"/>
-        </visual>
-        <collision>
-            <origin xyz="4.39926e-15 0.16 0.0115" rpy="-1.9984e-14 -1.5708 0" />
-            <geometry>
-                <mesh filename="package://arm/src/meshes/skf_7202.stl"/>
-            </geometry>
-            <material name="bearing_material"/>
-        </collision>
-        <visual>
-            <origin xyz="0 0 0.02" rpy="-1.5708 7.90622e-48 0" />
+            <origin xyz="0 0.16 0.0115" rpy="-0 -1.5708 0" />
+            <geometry>
+                <mesh filename="package://arm/src/meshes/skf_7202.stl"/>
+            </geometry>
+            <material name="bearing_material"/>
+        </visual>
+        <collision>
+            <origin xyz="0 0.16 0.0115" rpy="-0 -1.5708 0" />
+            <geometry>
+                <mesh filename="package://arm/src/meshes/skf_7202.stl"/>
+            </geometry>
+            <material name="bearing_material"/>
+        </collision>
+        <visual>
+            <origin xyz="6.93889e-18 0 0.02" rpy="-1.5708 -9.99986e-31 0" />
             <geometry>
                 <mesh filename="package://arm/src/meshes/fixing_shoulder_tree.stl"/>
@@ -371,5 +369,5 @@
         </visual>
         <collision>
-            <origin xyz="0 0 0.02" rpy="-1.5708 7.90622e-48 0" />
+            <origin xyz="6.93889e-18 0 0.02" rpy="-1.5708 -9.99986e-31 0" />
             <geometry>
                 <mesh filename="package://arm/src/meshes/fixing_shoulder_tree.stl"/>
@@ -378,37 +376,33 @@
         </collision>
         <visual>
-            <origin xyz="2.15453e-14 0.0969992 -0.033" rpy="1.5708 2.32728e-13 -3.14159" />
+            <origin xyz="6.47399e-15 0.0969992 -0.033" rpy="1.5708 1.1896e-13 3.14159" />
             <geometry>
                 <mesh filename="package://arm/src/meshes/xl430.stl"/>
             </geometry>
-            <material name="xl430_material">
-                <color rgba="0.501961 0.501961 0.501961 1.0"/>
-            </material>
-        </visual>
-        <collision>
-            <origin xyz="2.15453e-14 0.0969992 -0.033" rpy="1.5708 2.32728e-13 -3.14159" />
+            <material name="xl430_material"/>
+        </visual>
+        <collision>
+            <origin xyz="6.47399e-15 0.0969992 -0.033" rpy="1.5708 1.1896e-13 3.14159" />
             <geometry>
                 <mesh filename="package://arm/src/meshes/xl430.stl"/>
             </geometry>
-            <material name="xl430_material">
-                <color rgba="0.501961 0.501961 0.501961 1.0"/>
-            </material>
-        </collision>
-        <visual>
-            <origin xyz="1.41831e-14 -3.60822e-16 -0.076" rpy="1.5708 2.32728e-13 -3.14159" />
-            <geometry>
-                <mesh filename="package://arm/src/meshes/arm_elbow.stl"/>
-            </geometry>
-            <material name="pvc"/>
-        </visual>
-        <collision>
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