Commit message: rviz simulation

File: arm/src/urdf/robot.xacro (robot description, xacro)
@@ -1,883 +1,915 @@
 <robot xmlns:xacro="http://www.ros.org/wiki/xacro" name="Eden">
   <xacro:include filename="$(find arm)/src/urdf/materials.xacro" />
-<link name="reference">
-<origin xyz="0 0 0" rpy="0 0 0" />
-</link>
-  <joint name="fixed" type="fixed">
-    <parent link="reference"/>
-    <child link="base"/>
-  </joint>
-<link name="base">
-<visual>
-<origin xyz="-0.06 4.48374e-18 0.06" rpy="-3.14159 1.5708 0" />
-<geometry>
-<mesh filename="package://arm/src/meshes/skf_7208.stl"/>
-</geometry>
-<material name="bearing_material" />
-</visual>
-<collision>
-<origin xyz="-0.06 4.48374e-18 0.06" rpy="-3.14159 1.5708 0" />
-<geometry>
-<mesh filename="package://arm/src/meshes/skf_7208.stl"/>
-</geometry>
-<material name="bearing_material" />
-</collision>
-<visual>
-<origin xyz="0.0025 1.00198e-14 0.052" rpy="-1.5708 -0 1.5708" />
-<geometry>
-<mesh filename="package://arm/src/meshes/xl430.stl"/>
-</geometry>
-<material name="xl430_material">
-<color rgba="0.501961 0.501961 0.501961 1.0"/>
-</material>
-</visual>
-<collision>
-<origin xyz="0.0025 1.00198e-14 0.052" rpy="-1.5708 -0 1.5708" />
-<geometry>
-<mesh filename="package://arm/src/meshes/xl430.stl"/>
-</geometry>
-<material name="xl430_material">
-<color rgba="0.501961 0.501961 0.501961 1.0"/>
-</material>
-</collision>
-<visual>
-<origin xyz="0.00249985 1.45751e-07 0.088" rpy="3.14159 -0 -1.5708" />
-<geometry>
-<mesh filename="package://arm/src/meshes/small_gear_pilver.stl"/>
-</geometry>
-<material name="pvc" />
-</visual>
-<collision>
-<origin xyz="0.00249985 1.45751e-07 0.088" rpy="3.14159 -0 -1.5708" />
-<geometry>
-<mesh filename="package://arm/src/meshes/small_gear_pilver.stl"/>
-</geometry>
-<material name="pvc" />
-</collision>
-<visual>
-<origin xyz="-0.06 4.48374e-18 0.026" rpy="-0 1.5708 0" />
-<geometry>
-<mesh filename="package://arm/src/meshes/skf_7208.stl"/>
-</geometry>
-<material name="bearing_material" />
-</visual>
-<collision>
-<origin xyz="-0.06 4.48374e-18 0.026" rpy="-0 1.5708 0" />
-<geometry>
-<mesh filename="package://arm/src/meshes/skf_7208.stl"/>
-</geometry>
-<material name="bearing_material" />
-</collision>
-<visual>
-<origin xyz="0.00249985 1.45751e-07 0.082" rpy="0 -0 -1.5708" />
-<geometry>
-<mesh filename="package://arm/src/meshes/motor_link_xl.stl"/>
-</geometry>
-<material name="pla" />
-</visual>
-<collision>
-<origin xyz="0.00249985 1.45751e-07 0.082" rpy="0 -0 -1.5708" />
-<geometry>
-<mesh filename="package://arm/src/meshes/motor_link_xl.stl"/>
-</geometry>
-<material name="pla" />
-</collision>
-<visual>
-<origin xyz="0 0 0" rpy="0 -0 0" />
-<geometry>
-<mesh filename="package://arm/src/meshes/foundation.stl"/>
-</geometry>
-<material name="wood" />
-</visual>
-<collision>
-<origin xyz="0 0 0" rpy="0 -0 0" />
-<geometry>
-<mesh filename="package://arm/src/meshes/foundation.stl"/>
-</geometry>
-<material name="wood" />
-</collision>
-<visual>
-<origin xyz="-6.93889e-18 0.115 0" rpy="0 -0 1.48691e-16" />
-<geometry>
-<mesh filename="package://arm/src/meshes/wall_side.stl"/>
-</geometry>
-<material name="wood" />
-</visual>
-<collision>
-<origin xyz="-6.93889e-18 0.115 0" rpy="0 -0 1.48691e-16" />
-<geometry>
-<mesh filename="package://arm/src/meshes/wall_side.stl"/>
-</geometry>
-<material name="wood" />
-</collision>
-<visual>
-<origin xyz="0 0 0" rpy="0 -0 0" />
-<geometry>
-<mesh filename="package://arm/src/meshes/adapteur.stl"/>
-</geometry>
-<material name="pla" />
-</visual>
-<collision>
-<origin xyz="0 0 0" rpy="0 -0 0" />
-<geometry>
-<mesh filename="package://arm/src/meshes/adapteur.stl"/>
-</geometry>
-<material name="pla" />
-</collision>
-<visual>
-<origin xyz="-6.93889e-18 6.93889e-18 0" rpy="0 -0 1.48691e-16" />
-<geometry>
-<mesh filename="package://arm/src/meshes/wall_side.stl"/>
-</geometry>
-<material name="wood" />
-</visual>
-<collision>
-<origin xyz="-6.93889e-18 6.93889e-18 0" rpy="0 -0 1.48691e-16" />
-<geometry>
-<mesh filename="package://arm/src/meshes/wall_side.stl"/>
-</geometry>
-<material name="wood" />
-</collision>
-<visual>
-<origin xyz="-2.77556e-17 -6.93889e-18 -8.67362e-19" rpy="0 -0 0" />
-<geometry>
-<mesh filename="package://arm/src/meshes/wall_front.stl"/>
-</geometry>
-<material name="wood" />
-</visual>
-<collision>
-<origin xyz="-2.77556e-17 -6.93889e-18 -8.67362e-19" rpy="0 -0 0" />
-<geometry>
-<mesh filename="package://arm/src/meshes/wall_front.stl"/>
-</geometry>
-<material name="wood" />
-</collision>
-<visual>
-<origin xyz="0 0 0" rpy="0 -0 0" />
-<geometry>
-<mesh filename="package://arm/src/meshes/cover.stl"/>
-</geometry>
-<material name="wood" />
-</visual>
-<collision>
-<origin xyz="0 0 0" rpy="0 -0 0" />
-<geometry>
-<mesh filename="package://arm/src/meshes/cover.stl"/>
-</geometry>
-<material name="wood" />
-</collision>
-<inertial>
-<origin xyz="-0.0504246 -2.21857e-06 0.0403172" rpy="0 0 0"/>
-<mass value="1.76245" />
-<inertia ixx="0.0025824" ixy="2.14732e-07"  ixz="-2.84078e-05" iyy="0.00440605" iyz="1.21901e-07" izz="0.00562401" />
-</inertial>
-</link>
-<link name="hip">
-<visual>
-<origin xyz="7.70372e-34 0 0.062" rpy="3.14159 -0 -3.14088e-49" />
-<geometry>
-<mesh filename="package://arm/src/meshes/side_2.stl"/>
-</geometry>
-<material name="pvc" />
-</visual>
-<collision>
-<origin xyz="7.70372e-34 0 0.062" rpy="3.14159 -0 -3.14088e-49" />
-<geometry>
-<mesh filename="package://arm/src/meshes/side_2.stl"/>
-</geometry>
-<material name="pvc" />
-</collision>
-<visual>
-<origin xyz="-0.0235 -1.01238e-14 -0.116" rpy="3.14159 -0 -3.14088e-49" />
-<geometry>
-<mesh filename="package://arm/src/meshes/skf_7202.stl"/>
-</geometry>
-<material name="bearing_material" />
-</visual>
-<collision>
-<origin xyz="-0.0235 -1.01238e-14 -0.116" rpy="3.14159 -0 -3.14088e-49" />
-<geometry>
-<mesh filename="package://arm/src/meshes/skf_7202.stl"/>
-</geometry>
-<material name="bearing_material" />
-</collision>
-<visual>
-<origin xyz="7.70372e-34 0 0.062" rpy="3.14159 -0 -3.14088e-49" />
-<geometry>
-<mesh filename="package://arm/src/meshes/tree_base.stl"/>
-</geometry>
-<material name="pla" />
-</visual>
-<collision>
-<origin xyz="7.70372e-34 0 0.062" rpy="3.14159 -0 -3.14088e-49" />
-<geometry>
-<mesh filename="package://arm/src/meshes/tree_base.stl"/>
-</geometry>
-<material name="pla" />
-</collision>
-<visual>
-<origin xyz="-0.109 -4.69555e-14 -0.013" rpy="3.14159 -0 -3.14088e-49" />
-<geometry>
-<mesh filename="package://arm/src/meshes/big_gear_pilver.stl"/>
-</geometry>
-<material name="pvc" />
-</visual>
-<collision>
-<origin xyz="-0.109 -4.69555e-14 -0.013" rpy="3.14159 -0 -3.14088e-49" />
-<geometry>
-<mesh filename="package://arm/src/meshes/big_gear_pilver.stl"/>
-</geometry>
-<material name="pvc" />
-</collision>
-<visual>
-<origin xyz="0.0235 1.02626e-14 -0.116" rpy="3.14159 -0 -3.14088e-49" />
-<geometry>
-<mesh filename="package://arm/src/meshes/skf_7202.stl"/>
-</geometry>
-<material name="bearing_material" />
-</visual>
-<collision>
-<origin xyz="0.0235 1.02626e-14 -0.116" rpy="3.14159 -0 -3.14088e-49" />
-<geometry>
-<mesh filename="package://arm/src/meshes/skf_7202.stl"/>
-</geometry>
-<material name="bearing_material" />
-</collision>
-<visual>
-<origin xyz="0.009 -0.06775 -0.12275" rpy="1.5708 1.5708 0" />
-<geometry>
-<mesh filename="package://arm/src/meshes/xl430.stl"/>
-</geometry>
-<material name="xl430_material">
-<color rgba="0.501961 0.501961 0.501961 1.0"/>
-</material>
-</visual>
-<collision>
-<origin xyz="0.009 -0.06775 -0.12275" rpy="1.5708 1.5708 0" />
-<geometry>
-<mesh filename="package://arm/src/meshes/xl430.stl"/>
-</geometry>
-<material name="xl430_material">
-<color rgba="0.501961 0.501961 0.501961 1.0"/>
-</material>
-</collision>
-<visual>
-<origin xyz="7.70372e-34 0 0.062" rpy="3.14159 -0 -3.14088e-49" />
-<geometry>
-<mesh filename="package://arm/src/meshes/side.stl"/>
-</geometry>
-<material name="pvc" />
-</visual>
-<collision>
-<origin xyz="7.70372e-34 0 0.062" rpy="3.14159 -0 -3.14088e-49" />
-<geometry>
-<mesh filename="package://arm/src/meshes/side.stl"/>
-</geometry>
-<material name="pvc" />
-</collision>
-<visual>
-<origin xyz="-0.016 -0.13525 -0.12275" rpy="1.5708 4.57546e-16 1.5708" />
-<geometry>
-<mesh filename="package://arm/src/meshes/small_gear_shoulder.stl"/>
-</geometry>
-<material name="pvc" />
-</visual>
-<collision>
-<origin xyz="-0.016 -0.13525 -0.12275" rpy="1.5708 4.57546e-16 1.5708" />
-<geometry>
-<mesh filename="package://arm/src/meshes/small_gear_shoulder.stl"/>
-</geometry>
-<material name="pvc" />
-</collision>
-<visual>
-<origin xyz="7.70372e-34 0 0.062" rpy="3.14159 -0 -3.14088e-49" />
-<geometry>
-<mesh filename="package://arm/src/meshes/fixing_base_tree.stl"/>
-</geometry>
-<material name="pla" />
-</visual>
-<collision>
-<origin xyz="7.70372e-34 0 0.062" rpy="3.14159 -0 -3.14088e-49" />
-<geometry>
-<mesh filename="package://arm/src/meshes/fixing_base_tree.stl"/>
-</geometry>
-<material name="pla" />
-</collision>
-<inertial>
-<origin xyz="0.000625949 -0.0110014 -0.0532948" rpy="0 0 0"/>
-<mass value="0.680307" />
-<inertia ixx="0.00269833" ixy="1.85331e-05"  ixz="2.96121e-05" iyy="0.00248518" iyz="-0.000437423" izz="0.000819679" />
-</inertial>
-</link>
-<link name="humerus">
-<visual>
-<origin xyz="0 0 0.02" rpy="-1.5708 7.90622e-48 0" />
-<geometry>
-<mesh filename="package://arm/src/meshes/arm_elbow.stl"/>
-</geometry>
-<material name="pvc" />
-</visual>
-<collision>
-<origin xyz="0 0 0.02" rpy="-1.5708 7.90622e-48 0" />
-<geometry>
-<mesh filename="package://arm/src/meshes/arm_elbow.stl"/>
-</geometry>
-<material name="pvc" />
-</collision>
-<visual>
-<origin xyz="0 0 0.02" rpy="-1.5708 7.90622e-48 0" />
-<geometry>
-<mesh filename="package://arm/src/meshes/tree_shoulder.stl"/>
-</geometry>
-<material name="pla" />
-</visual>
-<collision>
-<origin xyz="0 0 0.02" rpy="-1.5708 7.90622e-48 0" />
-<geometry>
-<mesh filename="package://arm/src/meshes/tree_shoulder.stl"/>
-</geometry>
-<material name="pla" />
-</collision>
-<visual>
-<origin xyz="5.05151e-15 4.58366e-07 -0.008" rpy="-9.57715e-14 -2.09115e-13 -5.16254e-15" />
-<geometry>
-<mesh filename="package://arm/src/meshes/big_gear_shoulder.stl"/>
-</geometry>
-<material name="pvc" />
-</visual>
-<collision>
-<origin xyz="5.05151e-15 4.58366e-07 -0.008" rpy="-9.57715e-14 -2.09115e-13 -5.16254e-15" />
-<geometry>
-<mesh filename="package://arm/src/meshes/big_gear_shoulder.stl"/>
-</geometry>
-<material name="pvc" />
-</collision>
-<visual>
-<origin xyz="4.39926e-15 0.16 0.0115" rpy="-1.9984e-14 -1.5708 0" />
-<geometry>
-<mesh filename="package://arm/src/meshes/skf_7202.stl"/>
-</geometry>
-<material name="bearing_material" />
-</visual>
-<collision>
-<origin xyz="4.39926e-15 0.16 0.0115" rpy="-1.9984e-14 -1.5708 0" />
-<geometry>
-<mesh filename="package://arm/src/meshes/skf_7202.stl"/>
-</geometry>
-<material name="bearing_material" />
-</collision>
-<visual>
-<origin xyz="0 0 0.02" rpy="-1.5708 7.90622e-48 0" />
-<geometry>
-<mesh filename="package://arm/src/meshes/fixing_shoulder_tree.stl"/>
-</geometry>
-<material name="pla" />
-</visual>
-<collision>
-<origin xyz="0 0 0.02" rpy="-1.5708 7.90622e-48 0" />
-<geometry>
-<mesh filename="package://arm/src/meshes/fixing_shoulder_tree.stl"/>
-</geometry>
-<material name="pla" />
-</collision>
-<visual>
-<origin xyz="2.15453e-14 0.0969992 -0.033" rpy="1.5708 2.32728e-13 -3.14159" />
-<geometry>
-<mesh filename="package://arm/src/meshes/xl430.stl"/>
-</geometry>
-<material name="xl430_material">
-<color rgba="0.501961 0.501961 0.501961 1.0"/>
-</material>
-</visual>
-<collision>
-<origin xyz="2.15453e-14 0.0969992 -0.033" rpy="1.5708 2.32728e-13 -3.14159" />
-<geometry>
-<mesh filename="package://arm/src/meshes/xl430.stl"/>
-</geometry>
-<material name="xl430_material">
-<color rgba="0.501961 0.501961 0.501961 1.0"/>
-</material>
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
Commit message: report workspace

File: arm/src/urdf/robot.xacro (robot description, xacro)
@@ -164,7 +164,7 @@
         </collision>
         <inertial>
-            <origin xyz="-0.0504246 -2.21857e-06 0.0403172" rpy="0 0 0"/>
-            <mass value="1.76245" />
-            <inertia ixx="0.0025824" ixy="2.14732e-07"  ixz="-2.84078e-05" iyy="0.00440605" iyz="1.21901e-07" izz="0.00562401" />
+            <origin xyz="-0.04596 -3.09902e-06 0.0414358" rpy="0 0 0"/>
+            <mass value="1.26177" />
+            <inertia ixx="0.001588" ixy="1.973e-07"  ixz="8.28818e-07" iyy="0.00336754" iyz="1.17545e-07" izz="0.00393728" />
         </inertial>
     </link>
@@ -301,12 +301,12 @@
         </collision>
         <inertial>
-            <origin xyz="0.000625949 -0.0110014 -0.0532948" rpy="0 0 0"/>
-            <mass value="0.680307" />
-            <inertia ixx="0.00269833" ixy="1.85331e-05"  ixz="2.96121e-05" iyy="0.00248518" iyz="-0.000437423" izz="0.000819679" />
+            <origin xyz="0.000589843 -0.0157104 -0.0737648" rpy="0 0 0"/>
+            <mass value="0.468773" />
+            <inertia ixx="0.00169453" ixy="1.54024e-05"  ixz="1.84051e-05" iyy="0.00152219" iyz="-0.000280798" izz="0.000693306" />
         </inertial>
     </link>
     <link name="humerus">
         <visual>
-            <origin xyz="0 0 0.02" rpy="-1.5708 7.90622e-48 0" />
+            <origin xyz="0 0 0.04" rpy="-1.5708 7.90622e-48 0" />
             <geometry>
                 <mesh filename="package://arm/src/meshes/arm_elbow.stl"/>
@@ -315,5 +315,5 @@
         </visual>
         <collision>
-            <origin xyz="0 0 0.02" rpy="-1.5708 7.90622e-48 0" />
+            <origin xyz="0 0 0.04" rpy="-1.5708 7.90622e-48 0" />
             <geometry>
                 <mesh filename="package://arm/src/meshes/arm_elbow.stl"/>
@@ -396,5 +396,5 @@
         </collision>
         <visual>
-            <origin xyz="1.41831e-14 -3.60822e-16 -0.056" rpy="1.5708 2.32728e-13 -3.14159" />
+            <origin xyz="1.41831e-14 -3.60822e-16 -0.076" rpy="1.5708 2.32728e-13 -3.14159" />
             <geometry>
                 <mesh filename="package://arm/src/meshes/arm_elbow.stl"/>
@@ -403,5 +403,5 @@
         </visual>
         <collision>
-            <origin xyz="1.41831e-14 -3.60822e-16 -0.056" rpy="1.5708 2.32728e-13 -3.14159" />
+            <origin xyz="1.41831e-14 -3.60822e-16 -0.076" rpy="1.5708 2.32728e-13 -3.14159" />
             <geometry>
                 <mesh filename="package://arm/src/meshes/arm_elbow.stl"/>
@@ -452,7 +452,7 @@
         </collision>
         <inertial>
-            <origin xyz="-1.91915e-09 0.0765854 -0.0183109" rpy="0 0 0"/>
-            <mass value="0.410438" />
-            <inertia ixx="0.00212281" ixy="1.60796e-11"  ixz="-3.42603e-11" iyy="0.000426526" iyz="9.22129e-05" izz="0.00191415" />
+            <origin xyz="-1.2026e-09 0.079896 -0.0180401" rpy="0 0 0"/>
+            <mass value="0.390303" />
+            <inertia ixx="0.00200387" ixy="8.02765e-12"  ixz="-2.14145e-11" iyy="0.00041595" iyz="9.04428e-05" izz="0.00180475" />
         </inertial>
     </link>
@@ -589,7 +589,7 @@
         </collision>
         <inertial>
-            <origin xyz="-2.41779e-09 0.0753772 -0.0183786" rpy="0 0 0"/>
-            <mass value="0.416076" />
-            <inertia ixx="0.00205925" ixy="4.49005e-11"  ixz="-3.93973e-11" iyy="0.000369826" iyz="0.000285291" izz="0.00188503" />
+            <origin xyz="-1.50406e-09 0.0815245 -0.0176273" rpy="0 0 0"/>
+            <mass value="0.380955" />
+            <inertia ixx="0.00183593" ixy="2.2036e-11"  ixz="-2.38889e-11" iyy="0.000351507" iyz="0.000297264" izz="0.00167685" />
         </inertial>
     </link>
@@ -806,7 +806,7 @@
         </collision>
         <inertial>
-            <origin xyz="0.00248635 0.0745478 -0.0118851" rpy="0 0 0"/>
-            <mass value="0.300847" />
-            <inertia ixx="0.000794342" ixy="-9.01559e-06"  ixz="-1.05922e-06" iyy="0.000146324" iyz="-3.09085e-05" izz="0.000814276" />
+            <origin xyz="0.00426559 0.0751605 -0.0130646" rpy="0 0 0"/>
+            <mass value="0.16977" />
+            <inertia ixx="0.000439429" ixy="2.64382e-06"  ixz="-1.86798e-06" iyy="7.03996e-05" iyz="-3.26778e-05" izz="0.000448041" />
         </inertial>
     </link>
@@ -864,5 +864,5 @@
         </collision>
         <inertial>
-            <origin xyz="-8.13152e-20 4.68375e-17 -0.0015" rpy="0 0 0"/>
+            <origin xyz="1.0842e-19 4.85723e-17 -0.0015" rpy="0 0 0"/>
             <mass value="3.375e-05" />
             <inertia ixx="5.0625e-11" ixy="0"  ixz="1.4412e-40" iyy="5.0625e-11" iyz="0" izz="5.0625e-11" />

Commit message: rename stl

File: arm/src/urdf/robot.xacro (robot description, xacro)
@@ -175,5 +175,5 @@
             <origin xyz="-6.93889e-18 0 0.062" rpy="-3.14159 -0 4.01069e-70" />
             <geometry>
-                <mesh filename="package://arm/src/meshes/side_2.stl"/>
+                <mesh filename="package://arm/src/meshes/right_side.stl"/>
             </geometry>
             <material name="pvc"/>
@@ -182,5 +182,5 @@
             <origin xyz="-6.93889e-18 0 0.062" rpy="-3.14159 -0 4.01069e-70" />
             <geometry>
-                <mesh filename="package://arm/src/meshes/side_2.stl"/>
+                <mesh filename="package://arm/src/meshes/right_side.stl"/>
             </geometry>
             <material name="pvc"/>
@@ -259,5 +259,5 @@
             <origin xyz="0 0 0.062" rpy="-3.14159 -0 4.01069e-70" />
             <geometry>
-                <mesh filename="package://arm/src/meshes/side.stl"/>
+                <mesh filename="package://arm/src/meshes/left_side.stl"/>
             </geometry>
             <material name="pvc"/>
@@ -266,5 +266,5 @@
             <origin xyz="0 0 0.062" rpy="-3.14159 -0 4.01069e-70" />
             <geometry>
-                <mesh filename="package://arm/src/meshes/side.stl"/>
+                <mesh filename="package://arm/src/meshes/left_side.stl"/>
             </geometry>
             <material name="pvc"/>
